Commit message: 1. Launches iiwa through hitting 2. Adds object - box

File: object_models/box.urdf (robot description, URDF)
Before this commit: robot simple_box, 1 links, 0 joints
Links:
- link my_box: geometry collision box size=0.2 0.2 0.2; visual box size=0.2 0.2 0.2

Commit message: Basic hitting motion with passive DS in place
One video is uploaded too

File: object_models/box.urdf (robot description, URDF)
Before this commit: robot simple_box, 1 links, 0 joints
Links:
- link my_box: mass 1.0 -> 0.2; geometry collision box size=0.4 0.4 0.4; visual box size=0.4 0.4 0.4

Commit message: New version of Jari DS
Still currently the code is only in one file but now the position in line works better

File: object_models/box.urdf (robot description, URDF)
Before this commit: robot simple_box, 1 links, 0 joints
Links:
- link my_box: geometry collision box size=0.2 0.6 1.0; visual box size=0.2 0.6 1.0
