Commit message: running version of hitting - if want to reverse

File: object_models/big_box.urdf (robot description, URDF)
Before this commit: robot simple_box, 1 links, 0 joints
Links:
- removed link my_box
- added link big_box, mass 15; collision box size=1.6 0.8 0.5; visual box size=1.6 0.8 0.5

Commit message: changing in progress for actual robot

File: object_models/big_box.urdf (robot description, URDF)
Before this commit: robot big_box, 1 links, 0 joints
Links:
- link big_box: geometry collision box size=1.6 0.8 0.4; visual box size=1.6 0.8 0.4

Commit message: changing hitting to mimic real life

File: object_models/big_box.urdf (robot description, URDF)
Before this commit: robot big_box, 1 links, 0 joints
Links:
- link big_box: geometry collision box size=1.6 0.8 0.2; visual box size=1.6 0.8 0.2

File: object_models/box.urdf (robot description, URDF)
Before this commit: robot simple_box, 1 links, 0 joints
Links:
- link my_box: mass 0.2 -> 0.05

Commit message: hitting objects checkpoint 2

File: object_models/big_box.urdf (robot description, URDF)
Before this commit: robot big_box, 1 links, 0 joints
Links:
- link big_box: geometry collision box size=1.6 0.8 0.1; visual box size=1.6 0.8 0.2

Commit message: Changes for the initial HW experiments

File: object_models/big_box.urdf (robot description, URDF)
Before this commit: robot big_box, 1 links, 0 joints
Links:
- link big_box: geometry collision box size=0.8 1.6 0.2; visual box size=0.8 1.6 0.2

File: object_models/box.urdf (robot description, URDF)
Before this commit: robot simple_box, 1 links, 0 joints
Links:
- link my_box: geometry collision box size=0.23 0.26 0.26; visual box size=0.23 0.26 0.26

Commit message: flux DS implemented

File: object_models/big_box.urdf (robot description, URDF)
Before this commit: robot big_box, 1 links, 0 joints
Links:
- link big_box: geometry collision box size=0.8 1.6 0.1; visual box size=0.8 1.6 0.1

File: object_models/box.urdf (robot description, URDF)
Before this commit: robot simple_box, 1 links, 0 joints
Links:
- link my_box: geometry collision box size=0.23 0.26 0.4; visual box size=0.23 0.26 0.4
